File: STTS22H_Breakout_Board/STTS22H_Breakout_Board.sch (KiCad schematic (older format))
At the start: 4 parts, among them IC1 es_stts22h, J1 Conn_01x06_Female

Commit message: v1.0 finished.
Parts:
- IC1: footprint (none) -> EsLibs:STTS22H
- J1: footprint (none) -> Connector_PinHeader_2.54mm:PinHeader_1x06_P2.54mm_Vertical
- R1, R2: value R -> 4.7K; footprint (none) -> Resistor_SMD:R_0603_1608Metric
Changed lines of the file:
@@
 F 0 "IC1" H 4850 4350 50  0000 C CNN
 F 1 "es_stts22h" H 4850 4250 50  0000 C CNN
-F 2 "" H 5150 4100 50  0001 C CNN
+F 2 "EsLibs:STTS22H" H 5150 4100 50  0001 C CNN
 F 3 "https://www.st.com/resource/en/datasheet/stts22h.pdf" H 5150 4100 50  0001 C CNN
 	1    5150 4050
@@
 P 5400 3000
 F 0 "R2" H 5470 3046 50  0000 L CNN
-F 1 "R" H 5470 2955 50  0000 L CNN
-F 2 "" V 5330 3000 50  0001 C CNN
+F 1 "4.7K" H 5470 2955 50  0000 L CNN
+F 2 "Resistor_SMD:R_0603_1608Metric" V 5330 3000 50  0001 C CNN
 F 3 "~" H 5400 3000 50  0001 C CNN
 	1    5400 3000
@@
 P 5100 3000
 F 0 "R1" H 5170 3046 50  0000 L CNN
-F 1 "R" H 5170 2955 50  0000 L CNN
-F 2 "" V 5030 3000 50  0001 C CNN
+F 1 "4.7K" H 5170 2955 50  0000 L CNN
+F 2 "Resistor_SMD:R_0603_1608Metric" V 5030 3000 50  0001 C CNN
 F 3 "~" H 5100 3000 50  0001 C CNN
 	1    5100 3000
@@
 F 0 "J1" H 3750 3350 50  0000 L CNN
 F 1 "Conn_01x06_Female" H 3678 3435 50  0000 L CNN
-F 2 "" H 3650 3550 50  0001 C CNN
+F 2 "Connector_PinHeader_2.54mm:PinHeader_1x06_P2.54mm_Vertical" H 3650 3550 50  0001 C CNN
 F 3 "~" H 3650 3550 50  0001 C CNN
 	1    3650 3550
